File: Schematics/Programmer/Programmer.kicad_sch (KiCad schematic)
At the start: 17 parts, among them J1 USB_C_Receptacle_USB2.0, J2 SubModule, J3 I2C example, SW1 SEL_SEL, SW2 RESET, U1 AP2112K-3.3

Commit message: Programmer completed
Parts:
- removed J2: SubModule, Connector_PinHeader_2.54mm:PinHeader_2x06_P2.54mm_Vertical_SMD, symbol Connector:Conn_01x12_Female
- removed J3: I2C example, Connector_PinSocket_2.54mm:PinSocket_1x02_P2.54mm_Vertical, symbol Connector:Conn_01x02_Female
- removed SW1: SEL_SEL, Button_Switch_SMD:SW_DIP_SPSTx03_Slide_9.78x9.8mm_W8.61mm_P2.54mm, symbol Switch:SW_DIP_x03
- removed SW2: RESET, Button_Switch_SMD:SW_Push_SPST_NO_Alps_SKRK, symbol Switch:SW_SPST
- added C3, C4: 10uF, Capacitor_SMD:C_0603_1608Metric, symbol Device:C_Small
- added J2: J-link, Connector_PinSocket_1.27mm:PinSocket_2x05_P1.27mm_Vertical_SMD, symbol Connector_Generic:Conn_02x05_Odd_Even
- added J3: RJ12, Connector_RJ:RJ12_Amphenol_54601, symbol Connector:RJ12
- added Q1, Q2: DTC114T, libs:SOT346, symbol Transistor_BJT:DTC114T
- added R5: 10K, Resistor_SMD:R_0603_1608Metric, symbol Device:R_Small
- added SW1: ESP/SAMD, Button_Switch_THT:SW_CuK_JS202011CQN_DPDT_Straight, symbol Switch:SW_DPDT_x2
- added U2: CP2102N-A01-GQFN28, Package_DFN_QFN:QFN-28-1EP_5x5mm_P0.5mm_EP3.35x3.35mm, symbol Interface_USB:CP2102N-A01-GQFN28
- R2: value PullUp -> 22.1K
- R3: value PullUp -> 47.5K
- R4: value PullUp -> 1K
Connections:
- net SEL2 is gone; now on an unnamed net: R3.2
- net +3V3: now also C4.2, J2.1 (Pin_1), J3.2, R5.2, U2.6 (VDD), U2.7 (REGIN); no longer R2.1, R3.1
- net D+: now also U2.4 (D+)
- net D-: now also U2.5 (D-)
- net GND: now also R3.1, C3.2, C4.1, J2.3 (Pin_3), J3.4, U2.29 (GND), U2.3 (GND)
- net VBUS: now also R2.1
- net SEL1: no longer names the net of R2.2
- net SEL1: now also C3.1, U2.8 (VBUS)
- net SEL3: no longer names the net of R4.2
- net SEL3: now also U2.9 (~RSTb)
- new net: R5.1, U2.11 (~SUSPENDb)
- new net D0: J3.6, SW1.2 (B)
- new net D1: J3.5, SW1.5 (B)
- new net EN: Q2.3 (C), SW1.1 (A)
- new net IO0: Q1.3 (C), SW1.4 (A)
- new net RX: J3.3
- new net RXD: U2.25 (RXD)
- new net SWC: J2.4 (Pin_4), SW1.6 (C)
- new net SWD: J2.2 (Pin_2), SW1.3 (C)
- new net TX: J3.1
- new net TXD: U2.26 (TXD)
- new net ~DTR: Q1.2 (E), Q2.1 (B), U2.28 (~DTR)
- new net ~RTS: Q1.1 (B), Q2.2 (E), U2.24 (~RTS)
- no-connect marks 4 -> 25
Other:
- note added: "3.3V regulator"
- note added: "Auto Programmer"
- note added: "J-Link"
- note added: "Pogo programmer"
- note added: "USB"
- note added: "USB <-> TTL"
- title: (none) -> Programmer board
- moved on the sheet: C1, C2, D1, D2, D3, D4, D5, J1, R1, U1
