File: Schematics/TileBoard/TileBoard.kicad_pcb (KiCad board)
At the start: 0 parts

Commit message: TileBoard completed
Parts:
- added C1: 1uF, Capacitor_SMD:C_0603_1608Metric, F.Cu at (109.9, 77.1)
- added C2: 10uF, Capacitor_SMD:C_0603_1608Metric, F.Cu at (100.3, 74.9)
- added D1: APA102, LED_SMD:LED_RGB_5050-6, F.Cu at (98.8, 59.9)
- added J1: Input, Connector_PinSocket_2.54mm:PinSocket_1x05_P2.54mm_Vertical, F.Cu at (94.0, 64.6)
- added J2: Power, InvertedSwitch:Cherry_MX_PCB_Form, F.Cu at (108.1, 64.5)
- added J3: Output, Connector_PinSocket_2.54mm:PinSocket_1x05_P2.54mm_Vertical, F.Cu at (117.2, 64.6)
- added J4: Prog, Connector:Tag-Connect_TC2030-IDC-NL_2x03_P1.27mm_Vertical, F.Cu at (112.6, 80.6)
- added R1: 10k, Resistor_SMD:R_0603_1608Metric, F.Cu at (111.5, 77.1)
- added R2: 10k, Resistor_SMD:R_0603_1608Metric, F.Cu at (105.5, 63.5)
- added SW1: Mode, Button_Switch_SMD:SW_Push_SPST_NO_Alps_SKRK, F.Cu at (105.6, 60.7)
- added U1: ATSAMD21E18A-M, Package_DFN_QFN:QFN-32-1EP_5x5mm_P0.5mm_EP3.6x3.6mm, F.Cu at (105.4, 77.0)
Routing:
- net +3V3: track 0.00 -> 60.8 mm, vias 0 -> 5
- net GND: track 0.00 -> 43.5 mm, vias 0 -> 3
- net /I3: track 0.00 -> 35.0 mm, vias 0 -> 1
- net /O3: track 0.00 -> 27.0 mm, vias 0 -> 2
- net /Mode_SW: track 0.00 -> 23.9 mm, vias 0 -> 2
- net Net-(D1-Pad1): track 0.00 -> 20.6 mm, vias 0 -> 2
- net /O5: track 0.00 -> 19.1 mm, vias 0 -> 1
- net Net-(D1-Pad2): track 0.00 -> 18.9 mm, vias 0 -> 2
- net /O4: track 0.00 -> 18.7 mm, vias 0 -> 1
- net /I1: track 0.00 -> 17.8 mm
- net /O1: track 0.00 -> 17.0 mm, vias 0 -> 1
- net /I2: track 0.00 -> 14.6 mm
- net /O2: track 0.00 -> 13.2 mm, vias 0 -> 1
- net /I5: track 0.00 -> 11.2 mm
- net /SWC: track 0.00 -> 11.1 mm, vias 0 -> 2
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Other:
- board outline added: 27.1 x 26.9 mm
- copper layers 0 -> 2
