File: Schematics/MainBoard/MainBoard.kicad_pcb (KiCad board)
At the start: 2 copper layers, 250 x 120 mm, 48 parts, among them J1 USB_C_Receptacle_USB2.0, J2 SubModule 1, J3 SubModule 1, J4 SubModule 1, J5 SubModule 1, J6 SubModule 1, J7 SubModule 1, J8 SubModule 1, J9 SubModule 1, Q1 DTC114T, Q2 DTC114T, SW1 SW_Push, SW2 PROG, SW3 RESET, U1 CP2102N-A01-GQFN28, U2 ESP32-S2-WROVER, U3 TPS63001, U4 MCP73831-2-OT

Commit message: Finished circuit - pre mousebites
Parts:
- removed D2, D3: LESD5D5.0CT1G, Diode_SMD:D_SOD-523
- removed J9: SubModule 1, Connector_PinHeader_2.54mm:PinHeader_2x06_P2.54mm_Vertical_SMD
- removed Q1, Q2: DTC114T, libs:SOT346
- removed U1: CP2102N-A01-GQFN28, Package_DFN_QFN:QFN-28-1EP_5x5mm_P0.5mm_EP3.35x3.35mm
- added J11: Prog, Connector:Tag-Connect_TC2030-IDC-NL_2x03_P1.27mm_Vertical, F.Cu at (92.5, 4.40)
- added J12: OLED, Connector_PinHeader_2.00mm:PinHeader_1x04_P2.00mm_Vertical_SMD_Pin1Left, F.Cu at (29.1, 40.3)
- added R10: 2.4k, Resistor_SMD:R_0603_1608Metric, F.Cu at (96.1, -26.2)
- added R11: 2.4k, Resistor_SMD:R_0603_1608Metric, F.Cu at (106.8, -18.7)
- added R12: 47k, Resistor_SMD:R_0603_1608Metric, F.Cu at (115.7, 3.13)
- added R14: 47k, Resistor_SMD:R_0603_1608Metric, F.Cu at (90.8, -18.7)
- added R8: 100k, Resistor_SMD:R_0603_1608Metric, F.Cu at (120.9, 5.64)
- added R9: 100k, Resistor_SMD:R_0603_1608Metric, F.Cu at (86.2, 9.68)
- added SW4: Question, Rotary_Encoder:RotaryEncoder_Alps_EC11E-Switch_Vertical_H20mm, F.Cu at (61.1, 41.2)
- added SW5: PHB2UOATS1A, PHB2UOATS1A:PHB2UOATS1A, F.Cu at (55.6, 23.2)
- BT1, U2: moved to B.Cu
- C1, C3: value 10uF -> 10u
- J1: moved to F.Cu
- R1: value 22.1K -> 47k
- R2: value 47.5K -> 47k
- R3: value 1K -> 47k
- R4: value 10K -> 47k
- SW1: value SW_Push -> Time; footprint Button_Switch_SMD:SW_Push_SPST_NO_Alps_SKRK -> Rotary_Encoder:RotaryEncoder_Alps_EC11E-Switch_Vertical_H20mm
- moved J4 160.1 mm to (257.0, 108.1), turned to 90 degrees
- moved J6 149.2 mm to (257.0, 95.3), turned to 90 degrees
- moved J7 139.9 mm to (257.0, 82.4), turned to 90 degrees
- moved J2 132.5 mm to (257.0, 69.6), turned to 90 degrees
- moved L1 105.2 mm to (69.1, -6.65)
- moved J3 103.5 mm to (41.1, 66.1), turned to 90 degrees
- moved C11 103.2 mm to (68.3, -2.61)
- moved BT1 101.3 mm to (46.7, 23.3), turned to 180 degrees
- moved U3 100.5 mm to (91.3, -25.0)
- moved C8 99.7 mm to (88.1, -16.2)
- moved R4 99.6 mm to (92.1, -21.3)
- moved R7 99.0 mm to (84.1, -16.2)
- moved R6 97.3 mm to (100.1, -21.2)
- moved RPROG1 97.1 mm to (96.1, -21.2)
- moved C10 93.7 mm to (104.1, -26.2)
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Connections:
- net /Submodule connectors/I2C_SCL_IN renamed /IOBoard connectors/I2C_SCL_IN
- net /Submodule connectors/I2C_SDA_IN renamed /IOBoard connectors/I2C_SDA_IN
- C1 pad 1: Net-(C1-Pad1) -> +3V3
- C3 pad 1: GND -> +3V3
- C3 pad 2: +3V3 -> GND
- C4 pad 1: Net-(C4-Pad1) -> /BATT_SW
- DSTAT1 pad 5: unconnected-(DSTAT1-Pad5) -> (no net)
- DSTAT1 pad 6: unconnected-(DSTAT1-Pad6) -> (no net)
- J1 pad A5: unconnected-(J1-PadA5) -> (no net)
- J1 pad A6: /D+ -> (no net)
- J1 pad A7: /D- -> (no net)
- J1 pad A8: unconnected-(J1-PadA8) -> (no net)
- J1 pad B5: unconnected-(J1-PadB5) -> (no net)
- J1 pad B6: /D+ -> (no net)
- J1 pad B7: /D- -> (no net)
- J1 pad B8: unconnected-(J1-PadB8) -> (no net)
- J2 pad 10: /SMRST -> /RESET
- J2 pad 7: unconnected-(J2-Pad7) -> (no net)
- J2 pad 9: unconnected-(J2-Pad9) -> (no net)
- J3 pad 10: /SMRST -> /RESET
- J3 pad 7: unconnected-(J3-Pad7) -> (no net)
- J3 pad 9: unconnected-(J3-Pad9) -> (no net)
- J4 pad 10: /SMRST -> /RESET
- J4 pad 7: unconnected-(J4-Pad7) -> (no net)
- J4 pad 9: unconnected-(J4-Pad9) -> (no net)
- J5 pad 10: /SMRST -> /RESET
- J5 pad 7: unconnected-(J5-Pad7) -> (no net)
- J5 pad 9: unconnected-(J5-Pad9) -> (no net)
- J6 pad 10: /SMRST -> /RESET
- J6 pad 7: unconnected-(J6-Pad7) -> (no net)
- J6 pad 9: unconnected-(J6-Pad9) -> (no net)
- J7 pad 10: /SMRST -> /RESET
- J7 pad 7: unconnected-(J7-Pad7) -> (no net)
- J7 pad 9: unconnected-(J7-Pad9) -> (no net)
- J8 pad 10: /SMRST -> /RESET
- J8 pad 7: unconnected-(J8-Pad7) -> (no net)
- J8 pad 9: unconnected-(J8-Pad9) -> (no net)
- R1 pad 1: VBUS -> /Q_B
- R1 pad 2: Net-(C1-Pad1) -> +3V3
- R2 pad 1: GND -> /T_B
- R2 pad 2: Net-(C1-Pad1) -> +3V3
- R3 pad 1: +3V3 -> /Q_A
- R3 pad 2: Net-(R3-Pad2) -> +3V3
- R4 pad 1: Net-(R4-Pad1) -> /T_A
- R5 pad 2: Net-(C4-Pad1) -> /BATT_SW
- U2 pad 10: unconnected-(U2-Pad10) -> (no net)
- U2 pad 11: unconnected-(U2-Pad11) -> (no net)
- U2 pad 12: unconnected-(U2-Pad12) -> (no net)
- U2 pad 13: unconnected-(U2-Pad13) -> (no net)
- U2 pad 14: unconnected-(U2-Pad14) -> (no net)
- U2 pad 15: unconnected-(U2-Pad15) -> (no net)
- U2 pad 16: unconnected-(U2-Pad16) -> /T_A
- U2 pad 17: unconnected-(U2-Pad17) -> /T_B
- U2 pad 18: unconnected-(U2-Pad18) -> /T_SW
- U2 pad 19: unconnected-(U2-Pad19) -> /Q_A
- U2 pad 20: unconnected-(U2-Pad20) -> /Q_B
- U2 pad 21: unconnected-(U2-Pad21) -> /Q_SW
- U2 pad 22: unconnected-(U2-Pad22) -> (no net)
- U2 pad 23: unconnected-(U2-Pad23) -> (no net)
- U2 pad 24: unconnected-(U2-Pad24) -> (no net)
- U2 pad 25: unconnected-(U2-Pad25) -> (no net)
- U2 pad 27: unconnected-(U2-Pad27) -> (no net)
- U2 pad 28: unconnected-(U2-Pad28) -> (no net)
- U2 pad 29: unconnected-(U2-Pad29) -> /BATT_ref
- U2 pad 30: unconnected-(U2-Pad30) -> (no net)
- U2 pad 31: unconnected-(U2-Pad31) -> (no net)
- U2 pad 32: unconnected-(U2-Pad32) -> (no net)
- U2 pad 33: unconnected-(U2-Pad33) -> /OLED_SCL_I2C
- U2 pad 34: unconnected-(U2-Pad34) -> /OLED_SDA_I2C
- U2 pad 35: unconnected-(U2-Pad35) -> /STAT_LED_D
- U2 pad 36: unconnected-(U2-Pad36) -> /STAT_LED_C
- U2 pad 37: unconnected-(U2-Pad37) -> (no net)
- U2 pad 38: unconnected-(U2-Pad38) -> (no net)
- U2 pad 39: unconnected-(U2-Pad39) -> (no net)
- U2 pad 4: unconnected-(U2-Pad4) -> /D0
- U2 pad 40: unconnected-(U2-Pad40) -> (no net)
- U2 pad 5: unconnected-(U2-Pad5) -> /D1
- U2 pad 6: unconnected-(U2-Pad6) -> /RESET
- U2 pad 7: unconnected-(U2-Pad7) -> (no net)
- U2 pad 8: unconnected-(U2-Pad8) -> (no net)
- U2 pad 9: unconnected-(U2-Pad9) -> (no net)
- U3 pad 5: Net-(C4-Pad1) -> /BATT_SW
Other:
- board size 250 x 120 mm -> 257.9 x 120 mm
