File: Schematics/Mainboard/Power rails.kicad_sch (KiCad schematic)
At the start: 8 parts, among them J5 Prot in, J6 Prot out, J7 Power rail, J8 Power rail

Commit message: Added Mainboard rev 1.0
Parts:
- D1: footprint LED_SMD:LED_0603_1608Metric -> LED_SMD:LED_1206_3216Metric_Castellated; LCSC Part (none) -> C2286
- JP1, JP2: footprint Jumper:SolderJumper-2_P1.3mm_Bridged_Pad1.0x1.5mm -> Jumper:SolderJumper-2_P1.3mm_Open_Pad1.0x1.5mm
- R4: LCSC Part (none) -> C23032
Changed lines of the file:
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@@
+      (effects (font (size 1.27 1.27)) hide)
+    )
+    (property "LCSC Part" "C23032" (id 4) (at 34.29 52.705 90)
       (effects (font (size 1.27 1.27)) hide)
     )
@@
     (property "Reference" "D1" (id 0) (at 45.085 47.7224 0))
     (property "Value" "SHORT LED" (id 1) (at 45.085 50.4975 0))
-    (property "Footprint" "LED_SMD:LED_0603_1608Metric" (id 2) (at 45.085 52.705 90)
+    (property "Footprint" "LED_SMD:LED_1206_3216Metric_Castellated" (id 2) (at 45.085 52.705 90)
       (effects (font (size 1.27 1.27)) hide)
     )
     (property "Datasheet" "~" (id 3) (at 45.085 52.705 90)
+      (effects (font (size 1.27 1.27)) hide)
+    )
+    (property "LCSC Part" "C2286" (id 4) (at 45.085 52.705 0)
       (effects (font (size 1.27 1.27)) hide)
     )
@@
     (property "Reference" "JP1" (id 0) (at 40.005 60.9558 0))
     (property "Value" "3.3V Jumper" (id 1) (at 40.005 63.7309 0))
-    (property "Footprint" "Jumper:SolderJumper-2_P1.3mm_Bridged_Pad1.0x1.5mm" (id 2) (at 40.005 67.31 0)
+    (property "Footprint" "Jumper:SolderJumper-2_P1.3mm_Open_Pad1.0x1.5mm" (id 2) (at 40.005 67.31 0)
       (effects (font (size 1.27 1.27)) hide)
     )
@@
     (property "Reference" "JP2" (id 0) (at 40.005 70.4808 0))
     (property "Value" "GND Jumper" (id 1) (at 40.005 73.2559 0))
-    (property "Footprint" "Jumper:SolderJumper-2_P1.3mm_Bridged_Pad1.0x1.5mm" (id 2) (at 40.005 76.835 0)
+    (property "Footprint" "Jumper:SolderJumper-2_P1.3mm_Open_Pad1.0x1.5mm" (id 2) (at 40.005 76.835 0)
       (effects (font (size 1.27 1.27)) hide)
     )
