File: Schematics/Mainboard/Mainboard.kicad_sch (KiCad schematic)
At the start: 12 parts, among them J1 USB-C, J2 USB in, J3 USB out, J4 NFC Conn, SW1 RESET, U1 ESP32-WROOM-32

Commit message: Added Mainboard rev 1.0
Parts:
- removed J2: USB in, custom:PinSocket_1x06_P2.54mm_Vertical, symbol Connector:Conn_01x06_Male
- removed J3: USB out, custom:PinSocket_1x06_P2.54mm_Vertical, symbol Connector:Conn_01x06_Male
- added H1, H2, H3, H4: MountingHole, MountingHole:MountingHole_3.2mm_M3, symbol Mechanical:MountingHole
- added R31, R32: 5k1, Resistor_SMD:R_0603_1608Metric, symbol Device:R_Small
- C1, C3: LCSC Part (none) -> C14663
- C2: LCSC Part (none) -> C19702
- J1: LCSC Part C165948 -> C2835315
- R1, R2, R3: value 10K -> 10k; LCSC Part (none) -> C25804
- SW1: LCSC Part (none) -> C778181
- U1: LCSC Part (none) -> C473012
Connections:
- net GND: now also R31.2, R32.2
- net PN532 IRQ: now also U1.17 (SHD/SD2)
- net RGB B: now also U1.13 (IO14); no longer U1.14 (IO12)
- net RGB R: now also U1.14 (IO12); no longer U1.13 (IO14)
- net T_B: now also U1.8 (IO32); no longer U1.9 (IO33)
- net T_SW: now also U1.9 (IO33); no longer U1.8 (IO32)
- net at J1.A5 (CC1): now also R31.1
- net at J1.B5 (CC2): now also R32.1
- net PN532 RST0: no longer names the net of J4.8 (Pin_8)
- no-connect marks 18 -> 12
Other:
- added sheet USB-TTL (USB-TTL.kicad_sch)
- sheet Power management ports: added none; removed +3.3V, +BATT, GND, VBUS
- sheet User interface ports: added none; removed SUB RX, SUB TX
- note added: "Mounting holes"
- note removed: "USB-TTL module"
- moved on the sheet: J1
