File: Schematics/Mainboard/Power management.kicad_sch (KiCad schematic)
At the start: 9 parts, among them J10 CHG in, J11 Batt, J12 CHG out, J13 DC-DC in, J14 DC-DC out, Q1 AO3401A, SW2 SW_SPDT

Commit message: Added Mainboard rev 1.0
Parts:
- added C10, C9: 10u, Capacitor_SMD:C_0603_1608Metric, symbol Device:C_Small
- added D3: Red, LED_SMD:LED_1206_3216Metric_Castellated, symbol Device:LED_Small
- added D5: Gre, LED_SMD:LED_1206_3216Metric_Castellated, symbol Device:LED_Small
- added D6: Yel, LED_SMD:LED_1206_3216Metric_Castellated, symbol Device:LED_Small
- added J2: Pololu DC-DC, Connector_PinSocket_2.54mm:PinSocket_1x04_P2.54mm_Vertical, symbol Connector:Conn_01x04_Female
- added J9: Batt alt, Connector_PinSocket_2.54mm:PinSocket_1x02_P2.54mm_Vertical, symbol Connector:Conn_01x02_Female
- added JP5: SHDN, Jumper:SolderJumper-2_P1.3mm_Open_Pad1.0x1.5mm, symbol Device:Jumper_NO_Small
- added JP6: DC_DC, Jumper:SolderJumper-2_P1.3mm_Open_Pad1.0x1.5mm, symbol Device:Jumper
- added R20, R21, R22: 1k5, Resistor_SMD:R_0603_1608Metric, symbol Device:R_Small
- added R23, R24: 1k, Resistor_SMD:R_0603_1608Metric, symbol Device:R_Small
- added R25, R26: 10k, Resistor_SMD:R_0603_1608Metric, symbol Device:R_Small
- added U5: MCP73833, Package_SO:MSOP-10_3x3mm_P0.5mm, symbol Custom:MCP73833
- J11: footprint Connector_JST:JST_PH_S2B-PH-K_1x02_P2.00mm_Horizontal -> Connector_JST:JST_PH_S2B-PH-SM4-TB_1x02-1MP_P2.00mm_Horizontal; LCSC Part C173752 -> (none)
Connections:
- net +3V3: now also JP6.2; no longer J14.2 (Pin_2), J14.3 (Pin_3)
- net +BATT: now also C10.1, J9.2 (Pin_2), U5.10 (VBat), U5.9 (VBat); no longer J13.2 (Pin_2), J13.3 (Pin_3)
- net GND: now also C10.2, C9.2, J2.2 (Pin_2), J9.1 (Pin_1), JP5.1, R23.2, R24.2, R25.2, R26.2, U5.5 (VSS)
- net POWER_SW: now also J13.2 (Pin_2), J13.3 (Pin_3), J2.3 (Pin_3)
- net VBUS: now also C9.1, D3.2 (A), D5.2 (A), D6.2 (A), U5.1 (VDD), U5.2 (VDD)
- new net: D5.1 (K), R21.1
- new net: D6.1 (K), R20.1
- new net: D3.1 (K), R22.1
- new net: R22.2, U5.7 (~PG)
- new net: R20.2, U5.3 (STAT1)
- new net: R25.1, R26.1, U5.8 (THERM)
- new net: R21.2, U5.4 (STAT2)
- new net: J2.4 (Pin_4), JP5.2
- new net: R23.1, R24.1, U5.6 (PROG)
- new net DCDC: J14.2 (Pin_2), J14.3 (Pin_3), J2.1 (Pin_1), JP6.1
Other:
- note added: "PROG"
- note added: "THERM"
- moved on the sheet: D2, J10, J11, J12, Q1, R5, SW2
