File: Schematics/Mainboard/subModules/Wire tester/Wire tester.kicad_pcb (KiCad board)
At the start: 2 copper layers, 7 parts, among them J1 Input, Q1 SS8050

Commit message: added prelim wire tester
Parts:
- removed J1: Input, Connector_PinSocket_2.54mm:PinSocket_1x04_P2.54mm_Vertical
- added TP3: 3.3V Wire TP, TestPoint:TestPoint_Keystone_5015_Micro-Minature, B.Cu at (134.1, 85.1)
- added TP4: GND Wire TP, TestPoint:TestPoint_Keystone_5015_Micro-Minature, B.Cu at (128.5, 85.1)
- Q1, R1, R2: moved to B.Cu
- moved TP2 19.4 mm to (131.3, 113.8)
- moved R1 8.34 mm to (130.3, 97.8), turned to 180 degrees
- moved R2 7.69 mm to (132.6, 98.6), turned to -90 degrees
- moved TP1 7.59 mm to (131.3, 89.9)
- moved D1 5.21 mm to (130.0, 101.4)
- moved Q1 3.72 mm to (131.3, 104.9), turned to 90 degrees
Connections:
- Q1 pad 1: (no net) -> GND
Routing:
- net GND: track 0.00 -> 22.6 mm
- net +3V3: track 0.00 -> 14.8 mm
- net Net-(R1-Pad2): track 0.00 -> 8.68 mm, vias 0 -> 1
- net Net-(Q1-Pad2): track 0.00 -> 8.50 mm, vias 0 -> 1
- net Net-(D1-Pad1): track 0.00 -> 3.08 mm
- net Net-(D1-Pad2): track 0.00 -> 1.97 mm
Other:
- board outline added: 13.2 x 33.3 mm
